File: Hardware/OpenVault.kicad_pcb (KiCad board)
At the start: 2 copper layers, 45 x 54.7 mm, 45 parts, among them IC1 NPM1300-QEAA-R, IC2 STM32WB5MMGH6TR, IC3 TROPIC01, J03 HC-FPC-05-09-24RLTAG, J1 USB_C_Receptacle_USB2.0_16P, J2 Conn_01x02_Socket, J4 JUSHUO AFC01-S06FCC-00, J5 TC2030, Q1 Si1308EDL, SW2 SKSCLBE010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

Commit message: some hardware chagnes
Parts:
- added C17: 1uF/50V, Capacitor_SMD:C_0603_1608Metric, F.Cu at (129.0, 96.0)
- added C18: 1uF/50V, Capacitor_SMD:C_0603_1608Metric, F.Cu at (130.5, 96.0)
- added C19: 1uF/50V, Capacitor_SMD:C_0603_1608Metric, F.Cu at (132.0, 96.0)
- added C23: 1uF/50V, Capacitor_SMD:C_0603_1608Metric, F.Cu at (140.5, 96.0)
- added TP1: TestPoint, TestPoint:TestPoint_Pad_D1.0mm, F.Cu at (151.4, 105.1)
- added TP2: TestPoint, TestPoint:TestPoint_Pad_D1.0mm, F.Cu at (127.4, 90.7)
- added TP3: TestPoint, TestPoint:TestPoint_Pad_D1.0mm, F.Cu at (127.6, 81.9)
- added TP4: TestPoint, TestPoint:TestPoint_Pad_D1.0mm, F.Cu at (128.4, 119.0)
- added TP5: TestPoint, TestPoint:TestPoint_Pad_D1.0mm, F.Cu at (154.4, 81.9)
- added TP6: TestPoint, TestPoint:TestPoint_Pad_D1.0mm, F.Cu at (124.4, 119.0)
- added TP7: TestPoint, TestPoint:TestPoint_Pad_D1.0mm, F.Cu at (162.6, 82.5)
- added TP8: TestPoint, TestPoint:TestPoint_Pad_D1.0mm, F.Cu at (162.6, 80.3)
- added U3: W25Q128JVS, Package_SO:SOIC-8_5.3x5.3mm_P1.27mm, F.Cu at (122.0, 112.6)
- C8: value 4u7 -> 4u7/25V
- moved L1 141.7 mm to (131.8, 84.2), turned to 90 degrees
- moved IC1 131.8 mm to (136.9, 84.4)
- moved C5 130.7 mm to (129.9, 84.2), turned to 90 degrees
- moved C3 128.5 mm to (132.3, 82.0), turned to 180 degrees
- moved R1 126.2 mm to (139.3, 89.0), turned to -90 degrees
- moved C1 125.7 mm to (136.1, 89.1), turned to 90 degrees
- moved R5 118.8 mm to (125.9, 109.8), turned to 90 degrees
- moved C4 118.3 mm to (142.5, 84.7)
- moved C7 116.1 mm to (141.9, 83.5)
- moved C25 112.9 mm to (120.8, 107.3), turned to 180 degrees
- moved R6 106.8 mm to (162.3, 105.1), turned to 180 degrees
- moved R7 103.0 mm to (159.3, 105.1), turned to 180 degrees
- moved C6 102.4 mm to (143.0, 86.9), turned to -90 degrees
- moved TH1 100.8 mm to (145.5, 81.7), turned to 180 degrees
- moved C8 100.8 mm to (154.8, 109.0), turned to -90 degrees
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Connections:
- C8 pad 2: Net-(IC2-VBAT) -> GND
- IC2 pad 15: Net-(IC2-VBAT) -> +3V3
- IC2 pad 17: Net-(IC2-VBAT) -> +3V3
- IC2 pad 32: Net-(IC2-VBAT) -> +3V3
- IC2 pad 4: Net-(IC2-VBAT) -> +3V3
- IC2 pad 6: Net-(IC2-VBAT) -> +3V3
- J4 pad 1: GND -> I2C1_SDA
- J4 pad 2: TOUCH_INT -> I2C1_SCL
- J4 pad 3: TOUCH_RST -> +3V3
- J4 pad 4: +3V3 -> TOUCH_RST
- J4 pad 5: I2C1_SCL -> TOUCH_INT
- J4 pad 6: I2C1_SDA -> GND
- U1 pad 1: USBD- -> USBD+
- U1 pad 3: USBD+ -> USBD-
- U1 pad 4: P_USBD+ -> P_USBD-
- U1 pad 6: P_USBD- -> P_USBD+
Routing:
- net GND: track 0.00 -> 88.7 mm, vias 0 -> 181
- net MCU_SPI_MOSI: track 0.00 -> 69.2 mm, vias 0 -> 4
- net MCU_SPI_SCK: track 0.00 -> 67.3 mm, vias 0 -> 5
- net I2C1_SDA: track 0.00 -> 61.9 mm, vias 0 -> 2
- net MCU_SPI_MISO: track 0.00 -> 50.3 mm, vias 0 -> 2
- net I2C1_SCL: track 0.00 -> 49.0 mm, vias 0 -> 2
- net +3V3: track 0.00 -> 48.2 mm, vias 0 -> 30
- net DISPLAY_CSN: track 0.00 -> 44.9 mm, vias 0 -> 2
- net NPM_GPIO0: track 0.00 -> 44.1 mm, vias 0 -> 2
- net FLASH_CSN: track 0.00 -> 43.3 mm
- net SHPHLD: track 0.00 -> 39.9 mm
- net SWD_RESET: track 0.00 -> 39.8 mm, vias 0 -> 2
- net VBUS: track 0.00 -> 39.4 mm, vias 0 -> 5
- net P_USBD-: track 0.00 -> 36.4 mm
- net P_USBD+: track 0.00 -> 36.2 mm
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- added copper zone on F.Cu, net +3V3
- added copper zone on In2.Cu, net +3V3
- added copper zone on B.Cu, net GND
- added copper zone on F.Cu, net GND
- added copper zone on In1.Cu, net GND
Other:
- outline, holes or cut-outs redrawn
- copper layers 2 -> 4
- board text added: "Labs"
- board text added: "Nocta"
- board text added: "OpenVault V1"

Commit message: final before v2
Parts:
- moved L1 0.65 mm to (132.4, 84.3)
- moved R2 0.64 mm to (121.1, 103.5)
- moved C5 0.60 mm to (130.5, 84.2)
- moved Q1 0.54 mm to (124.0, 104.3)
- moved R3 0.54 mm to (121.1, 105.0)
Routing:
- net GND: track 88.7 -> 75.0 mm, vias 181 -> 140
- net I2C1_SDA: track 61.9 -> 49.5 mm
- net +3V3: track 48.2 -> 41.7 mm
- net DISPLAY_CSN: track 44.9 -> 43.8 mm, vias 2 -> 0
- net VSYS: track 26.7 -> 25.6 mm
- net MCU_SPI_SCK: track 67.3 -> 66.4 mm, vias 5 -> 3
- net Net-(D3-A): track 24.5 -> 23.7 mm, vias 2 -> 4
- net VBUS: track 39.4 -> 40.2 mm
- net Net-(IC1-SW2): track 2.98 -> 2.24 mm
- net /PREVGL: track 18.9 -> 19.5 mm
- net MCU_SPI_MOSI: track 69.2 -> 69.6 mm, vias 4 -> 2
