File: Hardware/OpenVault.kicad_sch (KiCad schematic)
At the start: 21 parts, among them IC1 STM32WB5MMG, IC2 NPM1300-QEAA-R7, J1 TYPE-C 16PIN 2MD(073), J2 SM02B-SRSS-TB_LF__SN_, SW1 SW_Push, U2 USBLC6-2SC6

Commit message: Working working
Parts:
- added C10, C14, C15, C16, C20, C21, C22, C9: 4u7/25V, symbol Device:C
- added C17, C18, C19, C23: 1uF/50V, symbol Device:C
- added D1, D2, D3: MBR0530, Diode_SMD:D_SOD-123, symbol Diode:MBR0530
- added J4: (no value), symbol OpenVaultSymbols:FPC6
- added J5: TC2030, Connector:Tag-Connect_TC2030-IDC-NL_2x03_P1.27mm_Vertical, symbol Connector:TC2030
- added L2: 10uH/1A, symbol Device:L
- added Q1: Si1308EDL, Package_TO_SOT_SMD:SOT-323_SC-70, symbol Transistor_FET:Si1308EDL
- added R2: 10K, symbol Device:R
- added R3: 0R47, symbol Device:R
- added R4: 3R, symbol Device:R
- renumbered C7 to C1, C9 to C11, C10 to C12, C11 to C13, C5 to C4, C6 to C5, C4 to C6, C1 to C7, IC2 to IC1, IC1 to IC2, U2 to U1
Connections:
- net +3V3: now also C17.2, C9.1, J4.4 (VDD), L2.1
- net GND: now also C14.2, C15.1, C16.1, C17.1, C18.1, C19.1, C20.1, C21.1, C22.1, C23.1, C9.2, D2.1 (K), J4.1 (GND), R2.2, R3.2, R4.1
- net I2C1_SCL: now also J4.5 (SCL)
- net I2C1_SDA: now also J4.6 (SDA)
- new net: C10.1, D1.1 (K), D2.2 (A)
- new net: C10.2, D3.2 (A), L2.2, Q1.3 (D)
- new net GDR_INK: Q1.1 (G), R2.1
- new net PREVGH: C14.1, D3.1 (K)
- new net PREVGL: C22.2, D1.2 (A)
- new net RESE_INK: Q1.2 (S), R3.1
- new net TOUCH_INT: J4.2 (INT)
- new net TOUCH_RST: J4.3 (RST)
- new net VCOM: C23.2
- no-connect marks 7 -> 10
Other:
- note added: "EINK DRIVER"
- note added: "EINK FPC"
- note added: "EINK TOUCH"

Commit message: tag connect
Connections:
- net TC_: now reaches J5.1
- net TC_: now also J5.2, J5.3, J5.4, J5.5, J5.6
Other:
- moved on the sheet: J5
Changed lines of the file:
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@@
 	)
 	(rectangle
+		(start 372.11 12.7)
+		(end 406.4 50.8)
+		(stroke
+			(width 0.254)
+			(type solid)
+		)
+		(fill
+			(type none)
+		)
+	)
+	(rectangle
 		(start 12.7 12.7)
 		(end 85.09 68.58)
@@
 		)
 	)
+	(global_label "TC_"
+		(shape bidirectional)
+		(at 382.27 35.56 180)
+		(fields_autoplaced yes)
+		(effects
+			(font
+				(size 0.889 0.889)
+			)
+			(justify right)
+		)
+		(property "Intersheetrefs" "${INTERSHEET_REFS}"
+			(at 377.159 35.56 0)
+			(hide yes)
+			(show_name no)
+			(do_not_autoplace no)
+			(effects
+				(font
+					(size 1.27 1.27)
+				)
+				(justify right)
+			)
+		)
+	)
 	(global_label "NPM_GPIO0"
 		(shape output)
@@
 		)
 	)
+	(global_label "TC_"
+		(shape bidirectional)
+		(at 382.27 38.1 180)
+		(fields_autoplaced yes)
+		(effects
+			(font
+				(size 0.889 0.889)
+			)
+			(justify right)
+		)
+		(property "Intersheetrefs" "${INTERSHEET_REFS}"
+			(at 377.159 38.1 0)
+			(hide yes)
+			(show_name no)
+			(do_not_autoplace no)
+			(effects
+				(font
+					(size 1.27 1.27)
+				)
+				(justify right)
+			)
+		)
+	)
+	(global_label "TC_"
+		(shape bidirectional)
+		(at 394.97 35.56 0)
+		(fields_autoplaced yes)
+		(effects
+			(font
+				(size 0.889 0.889)
+			)
+			(justify left)
+		)
+		(property "Intersheetrefs" "${INTERSHEET_REFS}"
+			(at 400.081 35.56 0)
+			(hide yes)
+			(show_name no)
+			(do_not_autoplace no)
+			(effects
+				(font
+					(size 1.27 1.27)
+				)
+				(justify left)
+			)
+		)
+	)
 	(global_label "P_USBD-"
 		(shape output)
@@
 		)
 	)
+	(global_label "TC_"
+		(shape bidirectional)
+		(at 394.97 40.64 0)
+		(fields_autoplaced yes)
+		(effects
+			(font
+				(size 0.889 0.889)
+			)
+			(justify left)
+		)
+		(property "Intersheetrefs" "${INTERSHEET_REFS}"
+			(at 400.081 40.64 0)
+			(hide yes)
+			(show_name no)
+			(do_not_autoplace no)
+			(effects
+				(font
+					(size 1.27 1.27)
+				)
+				(justify left)
+			)
+		)
+	)
 	(global_label "NTC"
 		(shape output)
@@
 		)
 	)
+	(global_label "TC_"
+		(shape bidirectional)
+		(at 394.97 38.1 0)
+		(fields_autoplaced yes)
+		(effects
+			(font
+				(size 0.889 0.889)
+			)
+			(justify left)
+		)
+		(property "Intersheetrefs" "${INTERSHEET_REFS}"
+			(at 400.081 38.1 0)
+			(hide yes)
+			(show_name no)
+			(do_not_autoplace no)
+			(effects
+				(font
+					(size 1.27 1.27)
+				)
+				(justify left)
+			)
+		)
+	)
 	(global_label "I2C1_SCL"
 		(shape bidirectional)
@@
 		)
 	)
+	(global_label "TC_"
+		(shape bidirectional)
+		(at 382.27 40.64 180)
+		(fields_autoplaced yes)
+		(effects
+			(font
+				(size 0.889 0.889)
+			)
+			(justify right)
+		)
+		(property "Intersheetrefs" "${INTERSHEET_REFS}"
+			(at 377.159 40.64 0)
+			(hide yes)
+			(show_name no)
+			(do_not_autoplace no)
+			(effects
+				(font
+					(size 1.27 1.27)
+				)
+				(justify right)
+			)
+		)
+	)
 	(global_label "SHPHLD"
 		(shape output)
@@
 	(symbol
 		(lib_id "Connector:TC2030")
-		(at 246.38 172.72 0)
+		(at 387.35 38.1 0)
 		(unit 1)
 		(body_style 1)
@@
 		(fields_autoplaced yes)
 		(property "Reference" "J5"
-			(at 247.65 160.02 0)
+			(at 387.3499 29.21 90)
 			(show_name no)
 			(do_not_autoplace no)
@@
 					(size 1.27 1.27)
 				)
+				(justify left)
 			)
 		)
 		(property "Value" "TC2030"
-			(at 247.65 162.56 0)
+			(at 389.8899 29.21 90)
 			(show_name no)
 			(do_not_autoplace no)
@@
 					(size 1.27 1.27)
 				)
+				(justify left)
 			)
 		)
 		(property "Footprint" "Connector:Tag-Connect_TC2030-IDC-NL_2x03_P1.27mm_Vertical"
-			(at 247.65 172.72 0)
+			(at 388.62 38.1 0)
 			(hide yes)
 			(show_name no)
@@
 		)
 		(property "Datasheet" "https://www.tag-connect.com/wp-content/uploads/bsk-pdf-manager/2019/12/TC2030-IDC-NL-Datasheet-Rev-B.pdf"
-			(at 247.65 172.72 0)
+			(at 388.62 38.1 0)
 			(hide yes)
 			(show_name no)
@@
 		)
 		(property "Description" "Tag-Connect’s 6-pins connector"
-			(at 246.38 172.72 0)
+			(at 387.35 38.1 0)
 			(hide yes)
 			(show_name no)

Commit message: all parts placed
Parts:
- added C24: 100nF, symbol Device:C
- added C25: 100n, symbol Device:C
- added R5: 10K, symbol Device:R
- added U2: W25Q128JVE, Package_SON:WSON-8-1EP_8x6mm_P1.27mm_EP3.4x4.3mm, symbol Memory_Flash:W25Q128JVE
Connections:
- net +3V3: now also J5.1, C25.1, R5.1, U2.3 (~{WP}/IO_{2}), U2.7 (~{HOLD}/~{RESET}/IO_{3}), U2.8 (VCC)
- net GND: now also J5.5, C24.2, C25.2, U2.4 (GND), U2.9 (EP)
- net MCU_SPI_CSN: now also R5.2, U2.1 (~{CS})
- net MCU_SPI_MISO: now also U2.2 (DO/IO_{1})
- net MCU_SPI_MOSI: now also U2.5 (DI/IO_{0})
- net MCU_SPI_SCK: now also U2.6 (CLK)
- net MCU_NRST renamed SWD_RESET
- net SWD_RESET: now also J5.3, C24.1
- removed net TC_: J5.1, J5.2, J5.3, J5.4, J5.5, J5.6
- new net SWD_CLK: J5.4
- new net SWD_IO: J5.2
- new net SWD_O: J5.6
- no-connect marks 10 -> 11
Other:
- note added: "TAG CONNECT SWD"
- moved on the sheet: J5

Commit message: lot of work
Parts:
- removed J2: SM02B-SRSS-TB_LF__SN_, SM02BSRSSTBLFSN, symbol SamacSys_Parts:SM02B-SRSS-TB_LF__SN_
- removed R4: 3R, symbol Device:R
- removed SW1: SW_Push, symbol Switch:SW_Push
- removed U2: W25Q128JVE, Package_SON:WSON-8-1EP_8x6mm_P1.27mm_EP3.4x4.3mm, symbol Memory_Flash:W25Q128JVE
- added FID1, FID2, FID3: Fiducial, symbol Mechanical:Fiducial
- added J2: Conn_01x02_Socket, Connector_JST:JST_PH_S2B-PH-SM4-TB_1x02-1MP_P2.00mm_Horizontal, symbol Connector:Conn_01x02_Socket
- added R6, R7: 4R7, Resistor_SMD:R_0603_1608Metric, symbol Device:R
- added R8: 10K, Resistor_SMD:R_0603_1608Metric, symbol Device:R
- added SW2: SKSCLBE010, :KEY-SMD_4P-SKSCLXX010, symbol OpenVaultSymbols:SKSCLBE010
- added TP1, TP2, TP3, TP4, TP5, TP6: TestPoint, symbol Connector:TestPoint
- added U3: W25Q128JVS, Package_SO:SOIC-8_5.3x5.3mm_P1.27mm, symbol Memory_Flash:W25Q128JVS
- C1, C3, C4, C5: footprint (none) -> Capacitor_SMD:C_0603_1608Metric; LCSC (none) -> C19702
- C10, C14, C15, C16, C20, C21, C22, C8, C9: footprint (none) -> Capacitor_SMD:C_0805_2012Metric; LCSC (none) -> C1779
- C11, C12, C13, C25: value 100n -> 100nF; footprint (none) -> Capacitor_SMD:C_0402_1005Metric; LCSC (none) -> C1525
- C17, C18, C19, C23: LCSC (none) -> C15849
- C2, C7: footprint (none) -> Capacitor_SMD:C_0402_1005Metric; LCSC (none) -> C52923
- C24: footprint (none) -> Capacitor_SMD:C_0402_1005Metric; LCSC (none) -> C1525
- C6: footprint (none) -> Capacitor_SMD:C_0603_1608Metric; LCSC (none) -> C23630
- D1, D2, D3: LCSC (none) -> C77336
- IC1: value NPM1300-QEAA-R7 -> NPM1300-QEAA-R; LCSC (none) -> C7466043
- IC2: value STM32WB5MMG -> STM32WB5MMGH6TR; LCSC (none) -> C5184586
- IC3: value (none) -> TROPIC01; now left out of the parts list
- J1: value TYPE-C 16PIN 2MD(073) -> USB_C_Receptacle_USB2.0_16P; MFPN TYPE-C 16PIN 2MD(073) -> (none); URL https://jlcpcb.com/partdetail/SHOUHAN-TYPE_C_16PIN_2MD_073/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 -> (none)
- J4: value (none) -> JUSHUO AFC01-S06FCC-00; footprint (none) -> OpenVaultFootprints:FPC-SMD_AFC01-S06FCC-00; LCSC (none) -> C262262
- L1: footprint (none) -> OpenVaultFootprints:IND-SMD_L2.0-W1.6; LCSC (none) -> C71386
- L2: value 10uH/1A -> 10uH1A; footprint (none) -> Inductor_SMD:L_Sunlord_SWPA4030S; LCSC (none) -> C38117
- Q1: LCSC (none) -> C7603347
- R1: footprint (none) -> Resistor_SMD:R_0603_1608Metric; LCSC (none) -> C23137
- R2, R5: footprint (none) -> Resistor_SMD:R_0603_1608Metric; LCSC (none) -> C25804
- R3: footprint (none) -> Resistor_SMD:R_0603_1608Metric; LCSC (none) -> C23411
- TH1: footprint (none) -> Inductor_SMD:L_0402_1005Metric; LCSC (none) -> C77131
- U1: LCSC (none) -> C2687116
Connections:
- net +3V3: now also R6.1, R7.2, TP4.1, U3.3 (~{WP}/IO_{2}), U3.7 (~{HOLD}/~{RESET}/IO_{3}), U3.8 (VCC)
- net BUSY: now also IC2.37 (PB14)
- net D/C: now also IC2.35 (PB13)
- net GND: now also J1.SH (SHIELD), J2.1 (Pin_1), R8.1, SW2.1, TP6.1, U3.4 (GND); no longer J1.S1 (SHIELD)
- net I2C1_SCL: now also IC2.14 (PB8), R6.2
- net I2C1_SDA: now also IC2.11 (PB9), R7.1
- net MCU_SPI_MISO: now also IC2.53 (PA6), U3.2 (DO/IO_{1})
- net MCU_SPI_MOSI: now also IC2.52 (PA7), U3.5 (DI/IO_{0})
- net MCU_SPI_SCK: now also IC2.54 (PA5), U3.6 (CLK)
- net NPM_GPIO0: now also IC2.39 (PB6)
- net P_USBD+: now also IC2.29 (PA12), U1.4 (I/O2); no longer U1.6 (I/O1)
- net P_USBD-: now also IC2.30 (PA11), U1.6 (I/O1); no longer U1.4 (I/O2)
- net RES: now also IC2.36 (PC6)
- net SHPHLD: now also SW2.3
- net SWD_CLK: now also IC2.26 (PA14)
- net SWD_IO: now also IC2.25 (PA13)
- net SWD_O: now also IC2.21 (PB3)
- net TOUCH_INT: now also IC2.24 (PC12)
- net TOUCH_RST: now also IC2.23 (PC11)
- net VBAT: now also J2.2 (Pin_2), TP5.1
- net VBUS: now also TP2.1
- net VSYS: now also IC1.1 (VOUT1), TP3.1
- net at IC2.13 (PH3-BOOT0): now also R8.2, TP1.1
- net FLASH_CSN: now reaches IC2.49 (PC4)
- net FLASH_CSN: now also R5.2, U3.1 (~{CS})
- net SECURE_CSN: now reaches IC2.50 (PA8)
- net SECURE_CSN: now also IC3.8 (SPI_CSN)
- net DISPLAY_CSN: now reaches IC2.51 (PA9)
- removed net MCU_SPI_CSN: IC3.8 (SPI_CSN), R5.2
- no-connect marks 11 -> 66
Other:
- note added: "EXTERNAL FLASH"
- note added: "Fiducials"
- note added: "Test Points"

Commit message: some hardware chagnes
Parts:
- removed FID1, FID2, FID3: Fiducial, symbol Mechanical:Fiducial
- added TP7, TP8: TestPoint, TestPoint:TestPoint_Pad_D1.0mm, symbol Connector:TestPoint
- C17, C18, C19, C23: footprint (none) -> Capacitor_SMD:C_0603_1608Metric
- C8: value 4u7 -> 4u7/25V
- IC3: now not fitted; now in the parts list
- R6, R7: value 4R7 -> 4.7K; LCSC C23164 -> C23162
- TP1, TP2, TP3, TP4, TP5, TP6: footprint (none) -> TestPoint:TestPoint_Pad_D1.0mm; now left out of the parts list
Connections:
- net +3V3: now also IC2.15 (VBAT), IC2.17 (VDDSMPS), IC2.32 (VDDUSB), IC2.4 (VREF), IC2.6 (VDDA), J4.3 (VDD); no longer J4.4 (VDD)
- net GND: now also C8.2, J4.6 (GND); no longer J4.1 (GND)
- net I2C1_SCL: now also J4.2 (SCL), TP8.1; no longer J4.5 (SCL)
- net I2C1_SDA: now also J4.1 (SDA), TP7.1; no longer J4.6 (SDA)
- net P_USBD+: now also U1.6 (I/O1); no longer U1.4 (I/O2)
- net P_USBD-: now also U1.4 (I/O2); no longer U1.6 (I/O1)
- net TOUCH_INT: now also J4.5 (INT); no longer J4.2 (INT)
- net TOUCH_RST: now also J4.4 (RST); no longer J4.3 (RST)
- net USBD+: now also U1.1 (I/O1); no longer U1.3 (I/O2)
- net USBD-: now also U1.3 (I/O2); no longer U1.1 (I/O1)
Other:
- note removed: "Fiducials"
- moved on the sheet: C24

Commit message: final before v2
Parts:
- L2: LCSC C38117 -> C497803
Changed lines of the file:
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@@
 			)
 		)
-		(property "LCSC" "C38117"
+		(property "LCSC" "C497803"
 			(at 251.46 76.2 90)
 			(hide yes)
