File: Hardware/OpenVault.kicad_sch (KiCad schematic)
At the start: 57 parts, among them IC1 NPM1300-QEAA-R, IC2 STM32WB5MMGH6TR, IC3 TROPIC01, J1 USB_C_Receptacle_USB2.0_16P, J2 Conn_01x02_Socket, J4 JUSHUO AFC01-S06FCC-00, J5 TC2030, Q1 Si1308EDL, SW2 SKSCLBE010, U1 USBLC6-2SC6, U3 W25Q128JVS

Commit message: Add VSON-8 3D model and production files
Add a STEP 3D model and KiCad footprint for the VSON-8 package, plus a Vias directory. Add production outputs (Hardware/production/V3.zip, V3_bom.csv, V3_designators.csv, V3_positions.csv) and update Hardware/production/netlist.ipc. Update KiCad project files (Hardware/OpenVault.kicad_pcb, .kicad_pro, .kicad_sch, and Symbols/OpenVaultSymbols.kicad_sym) and adjust fabrication-toolkit-options.json to include the new artifacts.
Parts:
- added C26: 4u7, Capacitor_SMD:C_0805_2012Metric, symbol Device:C
- added C27, C28: 22uF/25V, Capacitor_SMD:C_0805_2012Metric, symbol Device:C
- added L3: 2.2uH, OpenVaultFootprints:IND-SMD_L2.0-W1.6, symbol Device:L
- added R4: 267K, Resistor_SMD:R_0402_1005Metric, symbol Device:R
- added U2: TPS62840DLCR, VSON-8_L2.0-W1.5-P0.50-BL, symbol OpenVaultSymbols:TPS62840DLCR
Connections:
- net +3V3: no longer C17.2, C9.1, L2.1
- net BUSY: now also IC2.35 (PB13); no longer IC2.37 (PB14)
- net D/C: now also IC2.37 (PB14); no longer IC2.35 (PB13)
- net GND: now also C26.1, C27.2, C28.2, R4.2, U2.1 (GND), U2.3 (MODE), U2.6 (STOP)
- net P_USBD+: now also U1.4 (I/O2); no longer U1.6 (I/O1)
- net P_USBD-: now also U1.6 (I/O1); no longer U1.4 (I/O2)
- net USBD+: now also U1.3 (I/O2); no longer U1.1 (I/O1)
- net USBD-: now also U1.1 (I/O1); no longer U1.3 (I/O2)
- net VSYS: now also C26.2, U2.2 (VIN), U2.4 (EN)
- new net: L3.1, U2.7 (SW)
- new net: R4.1, U2.5 (VSET)
- new net +3V3_EINK: C17.2, C27.1, C28.1, C9.1, L2.1, L3.2, U2.8 (VOS)

Commit message: V4
Parts:
- removed J2: Conn_01x02_Socket, Connector_JST:JST_PH_S2B-PH-SM4-TB_1x02-1MP_P2.00mm_Horizontal, symbol Connector:Conn_01x02_Socket
- removed TH1: NTC 10K, Inductor_SMD:L_0402_1005Metric, symbol Device:Thermistor_NTC
- added J2: BATT_CON, Connector_JST:JST_SH_SM03B-SRSS-TB_1x03-1MP_P1.00mm_Horizontal, symbol Connector:Conn_01x03_Socket
- IC1: footprint QFN50P500X500X90-33N -> Package_DFN_QFN:QFN-32-1EP_5x5mm_P0.5mm_EP3.45x3.45mm_ThermalVias
- SW1: renamed from SW2; LCSC Part C115361 -> (none)
- U2: LCSC (none) -> C2071859
- renumbered C26 to C1, C7 to C10, C8 to C11, C24 to C12, C9 to C13, C10 to C14, C25 to C15, C11 to C16, C12 to C17, C13 to C18, C14 to C19, C1 to C2, C15 to C20, C16 to C21, C17 to C22, C19 to C23, C21 to C24, C22 to C25, C23 to C26, C20 to C27, C18 to C28, C2 to C3, C27 to C4, C3 to C5, C28 to C6, C4 to C7, C5 to C8, C6 to C9, J4 to J3, L3 to L1, L1 to L2, L2 to L3, R4 to R2, R8 to R3, R6 to R4, R7 to R5, R5 to R6, R2 to R7, R3 to R8, TP7 to TP3, TP8 to TP4, TP3 to TP5, TP4 to TP6, TP5 to TP7, TP6 to TP8
Connections:
- net GND: now also J2.1 (Pin_1)
- net NTC: now also J2.2 (Pin_2)
- net VBAT: now also J2.3 (Pin_3)
- net VSYS: no longer IC1.1 (VOUT1)
- no-connect marks 66 -> 67
